File: eagle/pogo_adapter_board_v1_1.brd (EAGLE design)
At the start: 101.6 x 81.3 mm, 38 parts, among them U1 ARDUINOR3-BPLACE

Commit message: redesign the pogo board not to hang silk screen off the edge of the board, since that makes seeed unhappy
Parts:
- U1: value ARDUINOR3-BPLACE -> ARDUINOR3; device adafruit:ARDUINOR3-BPLACE -> adafruit:ARDUINOR3-MINSHIELD
- moved U1 11.4 mm to (1.27, 0.00)
Changed lines of the file:
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@@
 <attribute name="TP_SIGNAL_NAME" value="" x="86.36" y="8.89" size="1.778" layer="28" rot="MR90" display="off"/>
 </element>
-<element name="U1" library="adafruit" package="ARDUINOR3-BPLACE" value="ARDUINOR3-BPLACE" x="-10.16" y="0"/>
+<element name="U1" library="adafruit" package="ARDUINOR3-MINSHIELD" value="ARDUINOR3" x="1.27" y="0" smashed="yes"/>
 <element name="PROGENABLE" library="SparkFun" package="JST-2-PTH-NS" value="" x="20.32" y="8.89" rot="R270"/>
 <element name="GO" library="SparkFun" package="JST-2-PTH-NS" value="" x="56.1594" y="66.294" rot="R90"/>
