File: eagle/pogo_adapter_board_v1_1.sch (EAGLE design)
At the start: 38 parts, among them U1 ARDUINOR3-BPLACE

Commit message: redesign the pogo board not to hang silk screen off the edge of the board, since that makes seeed unhappy
Parts:
- U1: value ARDUINOR3-BPLACE -> ARDUINOR3; device adafruit:ARDUINOR3-BPLACE -> adafruit:ARDUINOR3
Changed lines of the file:
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@@
 <part name="SEND_TEST" library="testpad" deviceset="PTR1" device="PAD1-13" value="PTR1PAD1-13"/>
 <part name="CONTACT" library="testpad" deviceset="PTR1" device="PAD1-13" value="PTR1PAD1-13"/>
-<part name="U1" library="adafruit" deviceset="ARDUINOR3" device="-BPLACE" value="ARDUINOR3-BPLACE"/>
+<part name="U1" library="adafruit" deviceset="ARDUINOR3" device="" value="ARDUINOR3"/>
 <part name="PROGENABLE" library="SparkFun" deviceset="M02" device="-JST-2-PTH-NO_SILK"/>
 <part name="GO" library="SparkFun" deviceset="M02" device="-JST-2-PTH-NO_SILK"/>
