File: eagle/massmfg_tinyx4_v1_1.brd (EAGLE design)
At the start: 76.2 x 76.2 mm, 30 parts, among them IC1 TINY24/44/84-SSU

Commit message: slight improvements to the lamp board
Parts:
- CONTACT, GND, LIGHT_TEST, MISO, MOSI, RESET, SCL, SEND_TEST, SPKR_TEST, V+: value PTR1PAD1-13 -> PTR1; device testpad:P1-13 -> testpad:P1-06
Other:
- board text added: "bryan duxbury 4/25/2013"
- board text added: "qmark lamp production v1.1.1"
- board text removed: "bryan duxbury 4/09/2013"
- board text removed: "qmark lamp production v1.1"
Changed lines of the file:
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@@
 <layer number="43" name="vRestrict" color="2" fill="10" visible="yes" active="yes"/>
 <layer number="44" name="Drills" color="7" fill="1" visible="no" active="yes"/>
-<layer number="45" name="Holes" color="7" fill="1" visible="no" active="yes"/>
+<layer number="45" name="Holes" color="7" fill="1" visible="yes" active="yes"/>
 <layer number="46" name="Milling" color="3" fill="1" visible="no" active="yes"/>
 <layer number="47" name="Measures" color="7" fill="1" visible="no" active="yes"/>
@@
 <text x="12.7" y="43.815" size="1.778" layer="25">SUPPLY</text>
 <text x="33.4518" y="19.4564" size="1.778" layer="25">XTAL</text>
-<text x="1.7526" y="72.6186" size="1.778" layer="25">qmark lamp production v1.1</text>
-<text x="1.5748" y="70.1294" size="1.778" layer="25">bryan duxbury 4/09/2013</text>
+<text x="1.7526" y="72.6186" size="1.778" layer="25">qmark lamp production v1.1.1</text>
+<text x="1.5748" y="70.1294" size="1.778" layer="25">bryan duxbury 4/25/2013</text>
 </plain>
 <attributes>
@@
 <element name="R6" library="resistor" package="M1206" value="15" x="43.18" y="68.58" rot="R270"/>
 <element name="LED4" library="smd_parts" package="OPTEK-DURIS5" value="" x="38.1" y="68.58"/>
-<element name="RESET" library="testpad" package="P1-13" value="PTR1PAD1-13" x="38.1" y="30.48" smashed="yes">
+<element name="RESET" library="testpad" package="P1-06" value="PTR1" x="38.1" y="30.48" smashed="yes">
 <attribute name="NAME" x="39.2082" y="27.7962" size="1.27" layer="25" rot="R45"/>
 <attribute name="VALUE" x="37.338" y="29.464" size="0.0254" layer="27"/>
-<attribute name="TP_SIGNAL_NAME" value="" x="38.1" y="27.94" size="1" layer="37"/>
-</element>
-<element name="MOSI" library="testpad" package="P1-13" value="PTR1PAD1-13" x="45.72" y="35.56" smashed="yes">
+</element>
+<element name="MOSI" library="testpad" package="P1-06" value="PTR1" x="45.72" y="35.56" smashed="yes">
 <attribute name="NAME" x="47.26" y="35.086" size="1.27" layer="25" rot="R45"/>
 <attribute name="VALUE" x="44.958" y="34.544" size="0.0254" layer="27"/>
-<attribute name="TP_SIGNAL_NAME" value="" x="45.72" y="33.02" size="1" layer="37"/>
-</element>
-<element name="MISO" library="testpad" package="P1-13" value="PTR1PAD1-13" x="45.72" y="40.64" smashed="yes">
+</element>
+<element name="MISO" library="testpad" package="P1-06" value="PTR1" x="45.72" y="40.64" smashed="yes">
 <attribute name="NAME" x="47.26" y="40.166" size="1.27" layer="25" rot="R45"/>
 <attribute name="VALUE" x="44.958" y="39.624" size="0.0254" layer="27"/>
-<attribute name="TP_SIGNAL_NAME" value="" x="45.72" y="38.1" size="1" layer="37"/>
-</element>
-<element name="SCL" library="testpad" package="P1-13" value="PTR1PAD1-13" x="45.72" y="45.72" smashed="yes">
+</element>
+<element name="SCL" library="testpad" package="P1-06" value="PTR1" x="45.72" y="45.72" smashed="yes">
 <attribute name="NAME" x="47.26" y="45.246" size="1.27" layer="25" rot="R45"/>
 <attribute name="VALUE" x="44.958" y="44.704" size="0.0254" layer="27"/>
-<attribute name="TP_SIGNAL_NAME" value="" x="45.72" y="43.18" size="1" layer="37"/>
 </element>
 <element name="R7" library="resistor" package="M1206" value="47" x="52.0954" y="67.691" smashed="yes" rot="R90">
@@
 </element>
 <element name="U$1" library="smd_parts" package="AWSCR-MG" value="AWSCR-MG" x="36" y="24"/>
-<element name="V+" library="testpad" package="P1-13" value="PTR1PAD1-13" x="30.48" y="30.48" smashed="yes">
+<element name="V+" library="testpad" package="P1-06" value="PTR1" x="30.48" y="30.48" smashed="yes">
 <attribute name="NAME" x="31.7406" y="28.1772" size="1.27" layer="25" rot="R45"/>
 <attribute name="VALUE" x="29.718" y="29.464" size="0.0254" layer="27"/>
-<attribute name="TP_SIGNAL_NAME" value="" x="30.48" y="27.94" size="1" layer="37"/>
 </element>
 <element name="R8" library="resistor" package="M1206" value="10M" x="46.99" y="25.4" smashed="yes" rot="R180">
@@
 <attribute name="VALUE" x="48.26" y="28.956" size="1.27" layer="27" rot="R180"/>
 </element>
-<element name="GND" library="testpad" package="P1-13" value="PTR1PAD1-13" x="30.48" y="45.72" smashed="yes">
+<element name="GND" library="testpad" package="P1-06" value="PTR1" x="30.48" y="45.72" smashed="yes">
 <attribute name="NAME" x="28.464" y="46.77" size="1.27" layer="25" rot="R45"/>
 <attribute name="VALUE" x="29.718" y="44.704" size="0.0254" layer="27"/>
-<attribute name="TP_SIGNAL_NAME" value="" x="30.48" y="43.18" size="1" layer="37"/>
 </element>
 <element name="U$3" library="smd_parts" package="10X3_CONNECTION_POINT" value="CONNECTION_POINT" x="17.78" y="34.29" rot="R90"/>
@@
 <element name="SPEAKER_PLUS" library="smd_parts" package="10X3_CONNECTION_POINT" value="CONNECTION_POINT" x="52.07" y="59.69"/>
 <element name="SPKR_MINUS" library="smd_parts" package="10X3_CONNECTION_POINT" value="CONNECTION_POINT" x="45.72" y="59.69"/>
-<element name="LIGHT_TEST" library="testpad" package="P1-13" value="PTR1PAD1-13" x="35.56" y="45.72" smashed="yes">
+<element name="LIGHT_TEST" library="testpad" package="P1-06" value="PTR1" x="35.56" y="45.72" smashed="yes">
 <attribute name="NAME" x="29.3784" y="41.1058" size="1.27" layer="25" rot="R45"/>
 <attribute name="VALUE" x="34.798" y="44.704" size="0.0254" layer="27"/>
-<attribute name="TP_SIGNAL_NAME" value="" x="35.56" y="43.18" size="1" layer="37"/>
-</element>
-<element name="SPKR_TEST" library="testpad" package="P1-13" value="PTR1PAD1-13" x="40.64" y="45.72" smashed="yes">
+</element>
+<element name="SPKR_TEST" library="testpad" package="P1-06" value="PTR1" x="40.64" y="45.72" smashed="yes">
 <attribute name="NAME" x="36.9139" y="43.5257" size="1.27" layer="25" rot="R45"/>
 <attribute name="VALUE" x="39.878" y="44.704" size="0.0254" layer="27"/>
-<attribute name="TP_SIGNAL_NAME" value="" x="40.64" y="43.18" size="1" layer="37"/>
-</element>
-<element name="SEND_TEST" library="testpad" package="P1-13" value="PTR1PAD1-13" x="45.72" y="30.48" smashed="yes">
+</element>
+<element name="SEND_TEST" library="testpad" package="P1-06" value="PTR1" x="45.72" y="30.48" smashed="yes">
 <attribute name="NAME" x="46.8028" y="30.9204" size="1.27" layer="25" rot="R45"/>
 <attribute name="VALUE" x="44.958" y="29.464" size="0.0254" layer="27"/>
-<attribute name="TP_SIGNAL_NAME" value="" x="45.72" y="27.94" size="1" layer="37"/>
-</element>
-<element name="CONTACT" library="testpad" package="P1-13" value="PTR1PAD1-13" x="30.48" y="38.1">
-<attribute name="TP_SIGNAL_NAME" value="" x="30.48" y="38.1" size="1.778" layer="27" display="off"/>
-</element>
+</element>
+<element name="CONTACT" library="testpad" package="P1-06" value="PTR1" x="30.48" y="38.1"/>
 </elements>
 <signals>
