File: eagle/massmfg_tinyx4_v1_1.sch (EAGLE design)
At the start: 30 parts, among them IC1 TINY24/44/84-SSU

Commit message: slight improvements to the lamp board
Parts:
- CONTACT, GND, LIGHT_TEST, MISO, MOSI, RESET, SCL, SEND_TEST, SPKR_TEST, V+: value PTR1PAD1-13 -> PTR1; device testpad:PTR1PAD1-13 -> testpad:PTR1
Changed lines of the file:
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@@
 <part name="GND3" library="supply1" deviceset="GNDA" device=""/>
 <part name="GND4" library="supply1" deviceset="GNDA" device=""/>
-<part name="RESET" library="testpad" deviceset="PTR1" device="PAD1-13" value="PTR1PAD1-13"/>
-<part name="MOSI" library="testpad" deviceset="PTR1" device="PAD1-13" value="PTR1PAD1-13"/>
-<part name="MISO" library="testpad" deviceset="PTR1" device="PAD1-13" value="PTR1PAD1-13"/>
-<part name="SCL" library="testpad" deviceset="PTR1" device="PAD1-13" value="PTR1PAD1-13"/>
+<part name="RESET" library="testpad" deviceset="PTR1" device="" value="PTR1"/>
+<part name="MOSI" library="testpad" deviceset="PTR1" device="" value="PTR1"/>
+<part name="MISO" library="testpad" deviceset="PTR1" device="" value="PTR1"/>
+<part name="SCL" library="testpad" deviceset="PTR1" device="" value="PTR1"/>
 <part name="P+4" library="supply1" deviceset="+5V" device=""/>
 <part name="R7" library="resistor" deviceset="R-US_" device="M1206" value="47"/>
 <part name="U$1" library="smd_parts" deviceset="AWSCR-MG" device=""/>
 <part name="P+5" library="supply1" deviceset="+5V" device=""/>
-<part name="V+" library="testpad" deviceset="PTR1" device="PAD1-13" value="PTR1PAD1-13"/>
+<part name="V+" library="testpad" deviceset="PTR1" device="" value="PTR1"/>
 <part name="R8" library="resistor" deviceset="R-US_" device="M1206" value="10M"/>
-<part name="GND" library="testpad" deviceset="PTR1" device="PAD1-13" value="PTR1PAD1-13"/>
+<part name="GND" library="testpad" deviceset="PTR1" device="" value="PTR1"/>
 <part name="GND5" library="supply1" deviceset="GNDA" device=""/>
 <part name="P+6" library="supply1" deviceset="+5V" device=""/>
@@
 <part name="SPEAKER_PLUS" library="smd_parts" deviceset="CONNECTION_POINT" device=""/>
 <part name="SPKR_MINUS" library="smd_parts" deviceset="CONNECTION_POINT" device=""/>
-<part name="LIGHT_TEST" library="testpad" deviceset="PTR1" device="PAD1-13" value="PTR1PAD1-13"/>
-<part name="SPKR_TEST" library="testpad" deviceset="PTR1" device="PAD1-13" value="PTR1PAD1-13"/>
-<part name="SEND_TEST" library="testpad" deviceset="PTR1" device="PAD1-13" value="PTR1PAD1-13"/>
-<part name="CONTACT" library="testpad" deviceset="PTR1" device="PAD1-13" value="PTR1PAD1-13"/>
+<part name="LIGHT_TEST" library="testpad" deviceset="PTR1" device="" value="PTR1"/>
+<part name="SPKR_TEST" library="testpad" deviceset="PTR1" device="" value="PTR1"/>
+<part name="SEND_TEST" library="testpad" deviceset="PTR1" device="" value="PTR1"/>
+<part name="CONTACT" library="testpad" deviceset="PTR1" device="" value="PTR1"/>
 <part name="GND6" library="supply1" deviceset="GNDA" device=""/>
 </parts>
