File: eagle/massmfg_tinyx4_v1_2.brd (EAGLE design)
At the start: 76.2 x 76.2 mm, 31 parts, among them IC1 TINY24/44/84-SSU

Commit message: latest updates to board based on EEs comments
Parts:
- removed R7: 47, resistor:M1206
- C1: device rcl:C1206 -> rcl:C0603
- moved R4 8.91 mm to (24.5, 53.4)
- moved R2 6.54 mm to (34.8, 56.5)
- moved C1 4.72 mm to (33.3, 38.1)
- moved LIGHT 4.70 mm to (29.6, 58.4)
- moved IC1 1.27 mm to (39.4, 38.1)
Connections:
- removed net N$17: R7.1, SPEAKER_PLUS.CONNECTION_POINT
- net +5V: now also SPEAKER_PLUS.CONNECTION_POINT; no longer R7.2
Routing:
- net N$2: track 47.1 -> 12.9 mm
- net N$4: track 36.3 -> 15.7 mm
- net LIGHT: track 10.3 -> 20.4 mm, vias 0 -> 2
- net SPKR: track 11.9 -> 20.0 mm, vias 0 -> 1
- net N$6: track 11.2 -> 3.60 mm
- net N$9: track 6.43 -> 13.1 mm, vias 0 -> 2
- net N$17: track 6.61 -> 0.00 mm
- net GNDA: track 100.7 -> 105.2 mm
- net +5V: track 163.0 -> 167.4 mm
- net N$18: track 154.1 -> 151.1 mm
- net N$13: track 3.84 -> 2.57 mm
- net N$14: track 3.84 -> 2.57 mm
- net RECV: track 13.5 -> 12.4 mm
- net SEND: track 14.6 -> 13.8 mm
- net N$12: track 5.02 -> 5.54 mm
Other:
- board text added: "bryan duxbury 8/1/2013"
- board text added: "qmark lamp production v1.2.2"
- board text removed: "bryan duxbury 7/23/2013"
- board text removed: "qmark lamp production v1.2"
