File: eagle/massmfg_tinyx4_v1_2.sch (EAGLE design)
At the start: 31 parts, among them IC1 TINY24/44/84-SSU

Commit message: latest updates to board based on EEs comments
Parts:
- removed R7: 47, resistor:R-US_M1206
- C1: device rcl:C-USC1206 -> rcl:C-USC0603
Connections:
- removed net N$17: R7.1, SPEAKER_PLUS.CONN
- net +5V: now also SPEAKER_PLUS.CONN; no longer R7.2
Changed lines of the file:
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@@
 <part name="SCL" library="testpad" deviceset="PTR1" device="" value="PTR1"/>
 <part name="P+4" library="supply1" deviceset="+5V" device=""/>
-<part name="R7" library="resistor" deviceset="R-US_" device="M1206" value="47"/>
 <part name="U$1" library="smd_parts" deviceset="AWSCR-MG" device=""/>
 <part name="P+5" library="supply1" deviceset="+5V" device=""/>
@@
 <part name="GND8" library="supply1" deviceset="GNDA" device=""/>
 <part name="P+7" library="supply1" deviceset="+5V" device=""/>
-<part name="C1" library="rcl" deviceset="C-US" device="C1206"/>
+<part name="C1" library="rcl" deviceset="C-US" device="C0603"/>
 </parts>
 <sheets>
@@
 <instance part="MISO" gate="G$1" x="71.12" y="43.18" rot="R90"/>
 <instance part="SCL" gate="G$1" x="71.12" y="40.64" rot="R90"/>
-<instance part="P+4" gate="1" x="160.02" y="104.14"/>
-<instance part="R7" gate="G$1" x="160.02" y="93.98" rot="R90"/>
+<instance part="P+4" gate="1" x="160.02" y="91.44"/>
 <instance part="U$1" gate="G$1" x="86.36" y="53.34"/>
 <instance part="P+5" gate="1" x="101.6" y="91.44"/>
@@
 </segment>
 <segment>
-<wire x1="160.02" y1="101.6" x2="160.02" y2="99.06" width="0.1524" layer="91"/>
-<pinref part="P+4" gate="1" pin="+5V"/>
-<pinref part="R7" gate="G$1" pin="2"/>
-</segment>
-<segment>
 <wire x1="101.6" y1="88.9" x2="101.6" y2="86.36" width="0.1524" layer="91"/>
 <wire x1="101.6" y1="86.36" x2="104.14" y2="86.36" width="0.1524" layer="91"/>
@@
 <wire x1="83.82" y1="99.06" x2="83.82" y2="101.6" width="0.1524" layer="91"/>
 </segment>
+<segment>
+<wire x1="160.02" y1="88.9" x2="160.02" y2="86.36" width="0.1524" layer="91"/>
+<wire x1="160.02" y1="86.36" x2="162.56" y2="86.36" width="0.1524" layer="91"/>
+<pinref part="SPEAKER_PLUS" gate="G$1" pin="CONN"/>
+<pinref part="P+4" gate="1" pin="+5V"/>
+</segment>
 </net>
 <net name="N$6" class="0">
@@
 </segment>
 </net>
-<net name="N$17" class="0">
-<segment>
-<wire x1="160.02" y1="88.9" x2="160.02" y2="86.36" width="0.1524" layer="91"/>
-<wire x1="160.02" y1="86.36" x2="162.56" y2="86.36" width="0.1524" layer="91"/>
-<pinref part="R7" gate="G$1" pin="1"/>
-<pinref part="SPEAKER_PLUS" gate="G$1" pin="CONN"/>
-</segment>
-</net>
